Commit message: add imu sensor

File: src/ugv_sim/scout/scout_description/urdf/scout_v2.xacro (robot description, xacro)
@@ -72,4 +72,39 @@
         <child link="inertial_link" />
     </joint>
+    <link name="imu_link">
+            <inertial>
+                <mass value="50" />
+                <!-- <mass value="50" /> -->
+                <!-- <origin xyz="-0.00065 -0.085 0.062" />
+                <inertia ixx="0.6022" ixy="-0.02364" ixz="-0.1197" iyy="1.7386" iyz="-0.001544" izz="2.0296" /> -->
+                <origin xyz="0.0 0.0 0.0" />
+                <inertia ixx="2.288641" ixy="0" ixz="0" iyy="5.103976" iyz="0" izz="3.431465" />
+            </inertial>
+        </link>
+        <gazebo reference="imu_link">
+            <gravity>true</gravity>
+            <sensor name="imu_sensor" type="imu">
+            <always_on>true</always_on>
+            <update_rate>100</update_rate>
+            <visualize>true</visualize>
+            <topic>imu_topic_name</topic>
+            <plugin filename="libgazebo_ros_imu_sensor.so" name="imu_plugin">
+                <topicName>imu</topicName>
+                <bodyName>imu_link</bodyName>
+                <updateRateHZ>10.0</updateRateHZ>
+                <gaussianNoise>0.0</gaussianNoise>
+                <xyzOffset>0 0 0</xyzOffset>
+                <rpyOffset>0 0 0</rpyOffset>
+                <frameName>imu_link</frameName>
+                <initialOrientationAsReference>false</initialOrientationAsReference>
+            </plugin>
+            <pose>0 0 0 0 0 0</pose>
+            </sensor>
+        </gazebo>
+        <joint name="imu_joint" type="fixed">
+            <origin xyz="0 0 0" rpy="0 0 0" />
+            <parent link="base_link" />
+            <child link="imu_link" />
+        </joint>
     <!-- For testing, hang the robot up in the air -->
     <!-- <link name="world" />

Commit message: added odom (world -> base_link publish) added uwb sensors, not yet functioning added new log data with correct frequencies issue: roslaunch not detecting rospy pakages

File: src/ugv_sim/scout/scout_description/urdf/scout_v2.xacro (robot description, xacro)
@@ -92,5 +92,5 @@
                 <topicName>imu</topicName>
                 <bodyName>imu_link</bodyName>
-                <updateRateHZ>10.0</updateRateHZ>
+                <updateRateHZ>100.0</updateRateHZ>
                 <gaussianNoise>0.0</gaussianNoise>
                 <xyzOffset>0 0 0</xyzOffset>
@@ -107,11 +107,4 @@
             <child link="imu_link" />
         </joint>
-    <!-- For testing, hang the robot up in the air -->
-    <!-- <link name="world" />
-    <joint name="world_to_base_link=" type="fixed">
-        <origin xyz="0 0 0.5" rpy="0 0 0" />
-        <parent link="world"/>
-        <child link="base_link"/>
-    </joint> -->
     <!-- Scout wheel macros -->
     <!-- wheel labeled from 0 to 3, conter-clockwise, starting from front right wheel -->

Commit message: added gps path follow (obstacle free) control node, not yet stable

File: src/ugv_sim/scout/scout_description/urdf/scout_v2.xacro (robot description, xacro)
@@ -58,9 +58,11 @@
 	    <frameId>base_link</frameId>
 	    <topicName>/gps/fix</topicName>
+          <referenceLatitude>31.0220344</referenceLatitude>
+          <referenceLongitude>121.4294481</referenceLongitude>
 	    <velocityTopicName>/gps/fix_velocity</velocityTopicName>
             <statusTopicName>/gps/status</statusTopicName>
 	    <offset>0 0 0</offset>
 	    <drift>0 0 0</drift>
-	    <gaussianNoise>0.05 0.05 0.05</gaussianNoise>
+	    <gaussianNoise>0.01 0.01 0.01</gaussianNoise>
 	    <velocityDrift>0.0001 0.0001 0.0001</velocityDrift>
 	    <velocityGaussianNoise>0.5 0.5 0.5</velocityGaussianNoise>
@@ -74,8 +76,5 @@
     <link name="imu_link">
             <inertial>
-                <mass value="50" />
-                <!-- <mass value="50" /> -->
-                <!-- <origin xyz="-0.00065 -0.085 0.062" />
-                <inertia ixx="0.6022" ixy="-0.02364" ixz="-0.1197" iyy="1.7386" iyz="-0.001544" izz="2.0296" /> -->
+                <mass value="20" />
                 <origin xyz="0.0 0.0 0.0" />
                 <inertia ixx="2.288641" ixy="0" ixz="0" iyy="5.103976" iyz="0" izz="3.431465" />
